Commit message: [Add] Fix some params

File: se2_navigation/car_demo/prius_description/urdf/prius.urdf (robot description, URDF)
Before this commit: robot prius, 28 links, 27 joints
Links:
- removed link back_camera_link
- removed link back_camera_link_optical
- removed link back_left_far_sonar_link
- removed link back_left_middle_sonar_link
- removed link back_right_far_sonar_link
- removed link back_right_middle_sonar_link
- removed link center_laser_link
- removed link front_camera_link
- removed link front_camera_link_optical
- removed link front_left_far_sonar_link
- removed link front_left_laser_link
- removed link front_left_middle_sonar_link
- removed link front_right_far_sonar_link
- removed link front_right_laser_link
- removed link front_right_middle_sonar_link
- removed link left_camera_link
- removed link left_camera_link_optical
- removed link right_camera_link
- removed link right_camera_link_optical
Joints:
- removed joint back_camera_joint
- removed joint back_camera_optical_joint
- removed joint back_left_far_sonar_joint
- removed joint back_left_middle_sonar_joint
- removed joint back_right_far_sonar_joint
- removed joint back_right_middle_sonar_joint
- removed joint center_laser_joint
- removed joint front_camera_joint
- removed joint front_camera_optical_joint
- removed joint front_left_far_sonar_joint
- removed joint front_left_laser_joint
- removed joint front_left_middle_sonar_joint
- removed joint front_right_far_sonar_joint
- removed joint front_right_laser_joint
- removed joint front_right_middle_sonar_joint
- removed joint left_camera_joint
- removed joint left_camera_optical_joint
- removed joint right_camera_joint
- removed joint right_camera_optical_joint
