Commit message: [Fix] Make wheel to move

File: se2_navigation/car_demo/erp42_description/urdf/erp42.urdf (robot description, URDF)
Before this commit: robot erp42, 8 links, 7 joints
Links:
- added link chassis, mass 160; collision box size=2.02 1.3 1.5; visual mesh filename=package://erp42_description/meshes/erp42_structure.dae scale=1 1 1
- link base_link: mass 160 -> 1; geometry 
- link front_left_wheel: mass 11 -> 5; geometry collision sphere length=0.15 radius=0.28; visual mesh filename=package://erp42_description/meshes/caucho.dae scale=1 1 1
- link front_right_wheel: mass 11 -> 5
- link rear_left_wheel: mass 11 -> 5
- link rear_right_wheel: mass 11 -> 5
Joints:
- added joint base_link_connection: type fixed, parent base_link, child chassis, origin xyz=0 0 0 rpy=0 0 0, axis 1 0 0
- joint front_left_steer_joint: parent base_link -> chassis
- joint front_left_wheel_joint: origin xyz=0 0 0 rpy=0 0 0 -> xyz=0 0 0 rpy=0 0 1.57
- joint front_right_steer_joint: parent base_link -> chassis
- joint front_right_wheel_joint: origin xyz=0 0 0 rpy=0 0 0 -> xyz=0 0 0 rpy=0 0 1.57
- joint rear_left_wheel_joint: origin xyz=-0.49 0.51 0 rpy=0 0 0 -> xyz=-0.49 0.51 0 rpy=0 0 1.57; parent base_link -> chassis
- joint rear_right_wheel_joint: origin xyz=-0.49 -0.51 0 rpy=0 0 0 -> xyz=-0.49 -0.51 0 rpy=0 0 1.57; parent base_link -> chassis
- joint steering_joint: origin xyz=0 0 0 rpy=0 0 0 -> xyz=0.357734 -0.627868 0.988243 rpy=-1.302101 0 0; parent base_link -> chassis

Commit message: [Fix] Fix some params

File: se2_navigation/car_demo/erp42_description/urdf/erp42.urdf (robot description, URDF)
Before this commit: robot erp42, 9 links, 8 joints
Links:
- link chassis: mass 160 -> 25; geometry collision box size=1.0 1.0 0.2; visual mesh filename=package://erp42_description/meshes/erp42_structure.dae scale=1 1 1

Commit message: [Fix] Fix many things

File: se2_navigation/car_demo/erp42_description/urdf/erp42.urdf (robot description, URDF)
Before this commit: robot erp42, 9 links, 8 joints
Joints:
- joint base_link_connection: origin xyz=0 0 0 rpy=0 0 0 -> xyz=0.2 0 -0.1 rpy=0 0 0
